Commit message: With out transition state

File: src/double_invert_pendulum_description/robot/visual/double_invert_pendulum.xacro (robot description, xacro)
@@ -7,18 +7,14 @@
     <!-- WORLD LINK (Fixed to ground) -->
     <link name="world"/>
-    <!-- FIXED JOINT (Base stuck to ground - no cart movement) -->
+    <!-- FIXED JOINT - RAISED TO PREVENT GROUND COLLISION -->
     <joint name="base" type="fixed">
         <parent link="world"/>
         <child link="base_link"/>
-        <origin xyz="0 0 0" rpy="0 0 0"/>  <!-- Base origin at ground level -->
+        <!-- Raised by 0.5m to keep pendulums above ground when hanging down -->
+        <origin xyz="0 0 0.5" rpy="0 0 0"/>
     </joint>
     <!-- BASE LINK -->
     <link name="base_link">
-        <!--
-          FIX: Using macro to calculate inertia from the mass variable
-          in pendulum_params.xacro and the collision box size.
-        -->
         <xacro:inertial_box mass="${mass_base}" x="0.25" y="0.15" z="0.18">
-            <!-- Origin from original URDF -->
             <origin xyz="4.35011143188239E-06 -4.26974202710915E-05 0.0926893522450359" rpy="0 0 0" />
         </xacro:inertial_box>
@@ -37,5 +33,5 @@
         </collision>
     </link>
-    <!-- REVOLUTE LINK (CONTINUOUS - unlimited rotation) -->
+    <!-- REVOLUTE LINK (ARM - CONTINUOUS ROTATION) -->
     <joint name="revolute_joint" type="continuous">
         <parent link="base_link"/>
@@ -47,11 +43,5 @@
     </joint>
     <link name="revolute_Link">
-        <!--
-          FIX: Using inertial_cylinder macro to calculate inertia based on
-          the '${mass_revolute}' variable from pendulum_params.xacro.
-          This replaces the hard-coded PDF values.
-        -->
         <xacro:inertial_cylinder mass="${mass_revolute}" length="0.05" radius="0.03">
-             <!-- Origin from SolidWorks PDF, converted to meters -->
             <origin xyz="-0.0393104703 -0.0011200394 -0.0049654099" rpy="0 0 0" />
         </xacro:inertial_cylinder>
@@ -80,10 +70,5 @@
     </joint>
     <link name="first_pendulum_link">
-        <!--
-          FIX: Using inertial_box macro to calculate inertia based on
-          the '${mass_pendulum1}' variable from pendulum_params.xacro.
-        -->
         <xacro:inertial_box mass="${mass_pendulum1}" x="0.02" y="0.14" z="0.02">
-            <!-- Origin from SolidWorks PDF, converted to meters -->
             <origin xyz="-0.0000001372 -0.0878320187 0.0001351167" rpy="0 0 0" />
         </xacro:inertial_box>
@@ -112,10 +97,5 @@
     </joint>
     <link name="second_pendulum_link">
-        <!--
-          FIX: Using inertial_box macro to calculate inertia based on
-          the '${mass_pendulum2}' variable from pendulum_params.xacro.
-        -->
         <xacro:inertial_box mass="${mass_pendulum2}" x="0.015" y="0.06" z="0.015">
-            <!-- Origin from SolidWorks PDF, converted to meters -->
             <origin xyz="-0.0000028766 -0.0299439674 0.001944771" rpy="0 0 0" />
         </xacro:inertial_box>

File: src/double_invert_pendulum_description/robot/visual/gazebo_full.xacro (robot description, xacro)
@@ -5,9 +5,8 @@
       <plugin>gz_ros2_control/GazeboSimSystem</plugin>
     </hardware>
-    <!-- Revolute joint control -->
     <joint name="revolute_joint">
       <command_interface name="effort">
-        <param name="min">-100</param>
-        <param name="max">100</param>
+        <param name="min">-50</param>
+        <param name="max">50</param>
       </command_interface>
       <state_interface name="position">
@@ -17,21 +16,19 @@
       <state_interface name="effort"/>
     </joint>
-    <!-- First pendulum joint control -->
     <joint name="first_pendulum_joint">
       <command_interface name="effort">
-        <param name="min">-100</param>
-        <param name="max">100</param>
+        <param name="min">-50</param>
+        <param name="max">50</param>
       </command_interface>
       <state_interface name="position">
-        <param name="initial_value"> 0.0 </param>
+        <param name="initial_value">0</param>
       </state_interface>
       <state_interface name="velocity"/>
       <state_interface name="effort"/>
     </joint>
-    <!-- Second pendulum joint control -->
     <joint name="second_pendulum_joint">
       <command_interface name="effort">
-        <param name="min">-100</param>
-        <param name="max">100</param>
+        <param name="min">-50</param>
+        <param name="max">50</param>
       </command_interface>
       <state_interface name="position">
@@ -44,7 +41,8 @@
   <gazebo>
     <plugin filename="gz_ros2_control-system" name="gz_ros2_control::GazeboSimROS2ControlPlugin">
+      <robot_param>robot_description</robot_param>
+      <robot_param_node>robot_state_publisher</robot_param_node>
       <parameters>$(find double_invert_pendulum_simulation)/config/controller_full.yaml</parameters>
     </plugin>
-    <!-- Sensor Manager (for IMU, Lidar, etc.) -->
     <plugin filename="libignition-gazebo-sensors-system.so"
             name="ignition::gazebo::systems::Sensors">
@@ -52,16 +50,3 @@
     </plugin>
   </gazebo>
-  <!-- Optional: IMU sensor on base_link -->
-  <!-- <gazebo reference="base_link">
-    <sensor name="imu_sensor" type="imu">
-      <always_on>true</always_on>
-      <update_rate>100.0</update_rate>
-      <visualize>true</visualize>
-      <topic>/imu/data</topic>
-      <gz_frame_id>base_link</gz_frame_id>
-      <plugin filename="libignition-gazebo-imu-system.so"
-              name="ignition::gazebo::systems::Imu"/>
-      <pose>0 0 0 0 0 0</pose>
-    </sensor>
-  </gazebo> -->
 </robot>

File: src/double_invert_pendulum_description/robot/visual/invert_pendulum_URDF.urdf (robot description, URDF)
Before this commit: robot inverted_pendulum_URDF, 4 links, 3 joints
Links:
- link base_link: geometry collision mesh filename=package://double_invert_pendulum_description/meshes/base_li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; visual mesh filename=package://double_invert_pendulum_description/meshes/base_li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
- link first_pendulum_link: mass 0.0997302210483473 -> 0.0997302210483471; geometry collision mesh filename=package://double_invert_pendulum_description/meshes/first_p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; visual mesh filename=package://double_invert_pendulum_description/meshes/first_p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
- link revolute_Link: mass 0.216240646404497 -> 0.22015507085087; geometry collision mesh filename=package://double_invert_pendulum_description/meshes/revolut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; visual mesh filename=package://double_invert_pendulum_description/meshes/revolut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
- link second_pendulum_link: mass 0.00680601326910171 -> 0.0733318769925464; geometry collision mesh filename=package://double_invert_pendulum_description/meshes/second_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; visual mesh filename=package://double_invert_pendulum_description/meshes/second_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
Joints:
- joint first_pendulum_joint: origin xyz=-0.107 -0.0002 0.023198 rpy=1.5708 0 -1.5708 -> xyz=-0.157 -0.0002 0.0232 rpy=1.5708 0 -1.5708
- joint second_pendulum_joint: origin xyz=0 -0.1432 0.0095 rpy=0 0 0 -> xyz=0 -0.1432 0.0135 rpy=0 0 0

File: src/double_invert_pendulum_description/robot/visual/pendulum_params.xacro (robot description, xacro)
@@ -3,34 +3,87 @@
     <!-- Constants -->
     <xacro:property name="PI" value="3.14159265359"/>
-    <!-- Joint positions from original URDF -->
+    <!-- ========================================== -->
+    <!-- JOINT POSITIONS (from inverted_pendulum_new.urdf) -->
+    <!-- ========================================== -->
+    <!-- Revolute joint (arm) position -->
     <xacro:property name="revolute_joint_x" value="0"/>
     <xacro:property name="revolute_joint_y" value="0"/>
     <xacro:property name="revolute_joint_z" value="0.2"/>
-    <xacro:property name="pendulum1_joint_x" value="-0.107"/>
+    <!-- First pendulum joint position -->
+    <xacro:property name="pendulum1_joint_x" value="-0.157"/>
     <xacro:property name="pendulum1_joint_y" value="-0.0002"/>
-    <xacro:property name="pendulum1_joint_z" value="0.023198"/>
+    <xacro:property name="pendulum1_joint_z" value="0.0232"/>
+    <!-- Second pendulum joint position -->
     <xacro:property name="pendulum2_joint_x" value="0"/>
     <xacro:property name="pendulum2_joint_y" value="-0.1432"/>
-    <xacro:property name="pendulum2_joint_z" value="0.0095"/>
-    <!--
-      Masses updated to match SolidWorks PDF reports (converted g -> kg)
-    -->
-    <xacro:property name="mass_base" value="0.5"/> <!-- Value from previous file, no PDF provided -->
-    <xacro:property name="mass_revolute" value="0.134003"/> <!-- 134.003 g -->
-    <xacro:property name="mass_pendulum1" value="0.050"/>    <!-- 50.0 g -->
-    <xacro:property name="mass_pendulum2" value="0.015"/>    <!-- 15.0 g -->
-    <!-- Joint limits - converted from continuous to revolute -->
-    <xacro:property name="joint_effort" value="100"/>
-    <xacro:property name="joint_velocity" value=" 50.0 "/>
-    <xacro:property name="joint_lower_limit" value="${-PI}"/>
-    <xacro:property name="joint_upper_limit" value="${PI}"/>
-    <!-- Joint dynamics - Revolute Joint -->
-    <xacro:property name="revolute_joint_damping" value="0.001"/>
-    <xacro:property name="revolute_joint_friction" value="0.02"/>
-    <!-- Joint dynamics - First Pendulum -->
-    <xacro:property name="first_pendulum_damping" value="0.001"/>
-    <xacro:property name="first_pendulum_friction" value="0.1"/>
-    <!-- Joint dynamics - Second Pendulum -->
-    <xacro:property name="second_pendulum_damping" value="0.001"/>
-    <xacro:property name="second_pendulum_friction" value="0.1"/>
+    <xacro:property name="pendulum2_joint_z" value="0.0135"/>
+    <!-- ========================================== -->
+    <!-- MASSES (from inverted_pendulum_new.urdf) -->
+    <!-- ========================================== -->
+    <xacro:property name="mass_base" value="0.951310569253784"/>
+    <xacro:property name="mass_revolute" value="0.22015507085087"/>
+    <xacro:property name="mass_pendulum1" value="0.190"/>  <!-- ~0.1 kg -->
+    <xacro:property name="mass_pendulum2" value="0.140"/>  <!-- ~0.073 kg -->
+    <!-- ========================================== -->
+    <!-- RESEARCH PAPER PARAMETERS -->
+    <!-- From "Transition Control of a Rotary Double Inverted Pendulum Using Direct Collocation" -->
+    <!-- ========================================== -->
+    <!-- Masses (for validation - should match above or be adjusted) -->
+    <xacro:property name="M1_paper" value="0.187"/>  <!-- First pendulum mass from paper -->
+    <xacro:property name="M2_paper" value="0.132"/>  <!-- Second pendulum mass from paper -->
+    <!-- Center of Mass Lengths -->
+    <xacro:property name="l1" value="0.072"/>   <!-- First pendulum CoM from pivot -->
+    <xacro:property name="l2" value="0.133"/>   <!-- Second pendulum CoM from pivot -->
+    <!-- Total Lengths -->
+    <xacro:property name="L1" value="0.1645"/>  <!-- First pendulum total length -->
+    <xacro:property name="R1" value="0.1625"/>  <!-- Arm radius -->
+    <xacro:property name="r1" value="0.1597"/>  <!-- Additional arm parameter -->
+    <xacro:property name="r2" value="0.0209"/>  <!-- Additional parameter -->
+    <!-- Inertias (kg·m²) from research paper -->
+    <xacro:property name="Ixx1" value="1.0415e-3"/>
+    <xacro:property name="Ixx2" value="8.8210e-4"/>
+    <xacro:property name="Iyy1" value="4.3569e-3"/>
+    <xacro:property name="Iyy2" value="4.9793e-3"/>
+    <xacro:property name="Izz1" value="3.3179e-3"/>
+    <xacro:property name="Izz2" value="4.8178e-3"/>
+    <xacro:property name="Ixz1" value="3.7770e-4"/>
+    <xacro:property name="Ixz2" value="1.9823e-4"/>
+    <!-- Friction coefficients from paper -->
+    <xacro:property name="c1_paper" value="2.41e-6"/>
+    <xacro:property name="c2_paper" value="1.09e-6"/>
+    <!-- ========================================== -->
+    <!-- JOINT LIMITS AND DYNAMICS -->
+    <!-- ========================================== -->
+    <!-- Joint effort and velocity limits -->
+    <xacro:property name="joint_effort" value="7.5"/>
+    <xacro:property name="joint_velocity" value="15.0"/>
+    <xacro:property name="joint_lower_limit" value="${-2*PI}"/>
+    <xacro:property name="joint_upper_limit" value="${2*PI}"/>
+    <!-- Revolute Joint (Arm) Dynamics - ACTUATED -->
+    <xacro:property name="revolute_joint_damping" value="${c1_paper}"/>
+    <xacro:property name="revolute_joint_friction" value="0.001"/>
+    <!-- First Pendulum Joint Dynamics - PASSIVE -->
+    <xacro:property name="first_pendulum_damping" value="${c1_paper}"/>
+    <xacro:property name="first_pendulum_friction" value="0.001"/>
+    <!-- Second Pendulum Joint Dynamics - PASSIVE -->
+    <xacro:property name="second_pendulum_damping" value="${c2_paper}"/>
+    <xacro:property name="second_pendulum_friction" value="0.001"/>
+    <!-- ========================================== -->
+    <!-- COLLISION GEOMETRY PARAMETERS -->
+    <!-- ========================================== -->
+    <!-- Base collision box -->
+    <xacro:property name="base_box_x" value="0.25"/>
+    <xacro:property name="base_box_y" value="0.15"/>
+    <xacro:property name="base_box_z" value="0.18"/>
+    <!-- Revolute link collision cylinder -->
+    <xacro:property name="revolute_radius" value="0.03"/>
+    <xacro:property name="revolute_length" value="0.05"/>
+    <!-- First pendulum collision box -->
+    <xacro:property name="pendulum1_box_x" value="0.02"/>
+    <xacro:property name="pendulum1_box_y" value="0.14"/>
+    <xacro:property name="pendulum1_box_z" value="0.02"/>
+    <!-- Second pendulum collision box -->
+    <xacro:property name="pendulum2_box_x" value="0.015"/>
+    <xacro:property name="pendulum2_box_y" value="0.11"/>
+    <xacro:property name="pendulum2_box_z" value="0.015"/>
 </robot>
